File: _autosave-TFG-PCB.sch (KiCad schematic (older format))
At the start: 14 parts

Commit message: Schematic created
Full implementation of the pcb schematic and annotation of its components
Parts:
- added D? (x4): SOD-123, symbol Device:D_Small
- added F?: 500mA, symbol Device:Polyfuse_Small
- added J?: TYPE-C-31-M-12, HRO_TYPE-C-31-M-12, symbol TYPE-C-31-M-12:TYPE-C-31-M-12
- added MX? (x4): MX-NoLED, symbol MX_Alps_Hybrid:MX-NoLED
- added R?: R_Small, symbol Device:R_Small
Connections:
- net labels added: COL0, COL1, ROW0, ROW1, VCC
- wire segments 45 -> 67
Changed lines of the file:
@@
 EESchema Schematic File Version 4
+LIBS:TFG-PCB-cache
 EELAYER 30 0
 EELAYER END
@@
 Text GLabel 1300 2650 0    50   Input ~ 0
 D-
+$Comp
+L TYPE-C-31-M-12:TYPE-C-31-M-12 J?
+U 1 1 6107DF22
+P 7050 1950
+F 0 "J?" H 7050 2617 50  0000 C CNN
+F 1 "TYPE-C-31-M-12" H 7050 2526 50  0000 C CNN
+F 2 "HRO_TYPE-C-31-M-12" H 7050 1950 50  0001 L BNN
+F 3 "" H 7050 1950 50  0001 L BNN
+F 4 "HRO Electronics" H 7050 1950 50  0001 L BNN "MANUFACTURER"
+F 5 "3.31mm" H 7050 1950 50  0001 L BNN "MAXIMUM_PACKAGE_HEIGHT"
+F 6 "Manufacturer Recommendations" H 7050 1950 50  0001 L BNN "STANDARD"
+F 7 "A" H 7050 1950 50  0001 L BNN "PARTREV"
+	1    7050 1950
+	1    0    0    -1
+$EndComp
+$Comp
+L Device:Polyfuse_Small F?
+U 1 1 6107EE6D
+P 8350 1550
+F 0 "F?" V 8145 1550 50  0000 C CNN
+F 1 "500mA" V 8236 1550 50  0000 C CNN
+F 2 "" H 8400 1350 50  0001 L CNN
+F 3 "~" H 8350 1550 50  0001 C CNN
+	1    8350 1550
+	0    1    1    0
+$EndComp
+$Comp
+L power:VCC #PWR?
+U 1 1 61080580
+P 8000 1550
+F 0 "#PWR?" H 8000 1400 50  0001 C CNN
+F 1 "VCC" H 8017 1723 50  0000 C CNN
+F 2 "" H 8000 1550 50  0001 C CNN
+F 3 "" H 8000 1550 50  0001 C CNN
+	1    8000 1550
+	1    0    0    -1
+$EndComp
+$Comp
+L power:+5V #PWR?
+U 1 1 610810C0
+P 8600 1550
+F 0 "#PWR?" H 8600 1400 50  0001 C CNN
+F 1 "+5V" H 8615 1723 50  0000 C CNN
+F 2 "" H 8600 1550 50  0001 C CNN
+F 3 "" H 8600 1550 50  0001 C CNN
+	1    8600 1550
+	1    0    0    -1
+$EndComp
+Wire Wire Line
+	7750 1550 8000 1550
+Wire Wire Line
+	8000 1550 8250 1550
+Connection ~ 8000 1550
+Wire Wire Line
+	8450 1550 8600 1550
+$Comp
+L power:GND #PWR?
+U 1 1 61084E96
+P 7900 2350
+F 0 "#PWR?" H 7900 2100 50  0001 C CNN
+F 1 "GND" H 7905 2177 50  0000 C CNN
+F 2 "" H 7900 2350 50  0001 C CNN
+F 3 "" H 7900 2350 50  0001 C CNN
+	1    7900 2350
+	1    0    0    -1
+$EndComp
+Wire Wire Line
+	7750 2350 7900 2350
+Text GLabel 6050 1850 0    50   Input ~ 0
+D+
+Text GLabel 6050 1950 0    50   Input ~ 0
+D-
+Text GLabel 8450 1950 2    50   Input ~ 0
+D+
+Text GLabel 8450 1850 2    50   Input ~ 0
+D-
+Wire Wire Line
+	7750 1850 8450 1850
+Wire Wire Line
+	7750 1950 8450 1950
+Wire Wire Line
+	6350 1850 6050 1850
+Wire Wire Line
+	6350 1950 6050 1950
+$Comp
+L Device:R_Small R?
+U 1 1 6108B301
+P 8000 2050
+F 0 "R?" V 7804 2050 50  0000 C CNN
+F 1 "R_Small" V 7895 2050 50  0000 C CNN
+F 2 "" H 8000 2050 50  0001 C CNN
+F 3 "~" H 8000 2050 50  0001 C CNN
+	1    8000 2050
+	0    1    1    0
+$EndComp
+Wire Wire Line
+	7750 2050 7900 2050
+$Comp
+L power:GND #PWR?
+U 1 1 6108CB90
+P 8250 2050
+F 0 "#PWR?" H 8250 1800 50  0001 C CNN
+F 1 "GND" H 8255 1877 50  0000 C CNN
+F 2 "" H 8250 2050 50  0001 C CNN
+F 3 "" H 8250 2050 50  0001 C CNN
+	1    8250 2050
+	1    0    0    -1
+$EndComp
+Wire Wire Line
+	8100 2050 8250 2050
+$Comp
+L MX_Alps_Hybrid:MX-NoLED MX?
+U 1 1 6108EC4B
+P 7600 3400
+F 0 "MX?" H 7633 3623 60  0000 C CNN
+F 1 "MX-NoLED" H 7633 3549 20  0000 C CNN
+F 2 "" H 6975 3375 60  0001 C CNN
+F 3 "" H 6975 3375 60  0001 C CNN
+	1    7600 3400
+	1    0    0    -1
+$EndComp
+$Comp
+L Device:D_Small D?
+U 1 1 6108F30D
+P 7300 3650
+F 0 "D?" V 7346 3582 50  0000 R CNN
+F 1 "SOD-123" V 7255 3582 50  0000 R CNN
+F 2 "" V 7300 3650 50  0001 C CNN
+F 3 "~" V 7300 3650 50  0001 C CNN
+	1    7300 3650
+	0    -1   -1   0
+$EndComp
+Wire Wire Line
+	7550 3550 7300 3550
+$Comp
+L MX_Alps_Hybrid:MX-NoLED MX?
+U 1 1 6109812B
+P 8350 3400
+F 0 "MX?" H 8383 3623 60  0000 C CNN
+F 1 "MX-NoLED" H 8383 3549 20  0000 C CNN
+F 2 "" H 7725 3375 60  0001 C CNN
+F 3 "" H 7725 3375 60  0001 C CNN
+	1    8350 3400
+	1    0    0    -1
+$EndComp
+$Comp
+L Device:D_Small D?
+U 1 1 61098131
+P 8050 3650
+F 0 "D?" V 8096 3582 50  0000 R CNN
+F 1 "SOD-123" V 8005 3582 50  0000 R CNN
+F 2 "" V 8050 3650 50  0001 C CNN
+F 3 "~" V 8050 3650 50  0001 C CNN
+	1    8050 3650
+	0    -1   -1   0
+$EndComp
+Wire Wire Line
+	8300 3550 8050 3550
+$Comp
+L MX_Alps_Hybrid:MX-NoLED MX?
+U 1 1 6109C001
+P 7600 4150
+F 0 "MX?" H 7633 4373 60  0000 C CNN
+F 1 "MX-NoLED" H 7633 4299 20  0000 C CNN
+F 2 "" H 6975 4125 60  0001 C CNN
+F 3 "" H 6975 4125 60  0001 C CNN
+	1    7600 4150
+	1    0    0    -1
+$EndComp
+$Comp
+L Device:D_Small D?
+U 1 1 6109C007
+P 7300 4400
+F 0 "D?" V 7346 4332 50  0000 R CNN
+F 1 "SOD-123" V 7255 4332 50  0000 R CNN
+F 2 "" V 7300 4400 50  0001 C CNN
+F 3 "~" V 7300 4400 50  0001 C CNN
+	1    7300 4400
+	0    -1   -1   0
+$EndComp
+Wire Wire Line
+	7550 4300 7300 4300
+$Comp
+L MX_Alps_Hybrid:MX-NoLED MX?
+U 1 1 6109C00E
+P 8350 4150
+F 0 "MX?" H 8383 4373 60  0000 C CNN
+F 1 "MX-NoLED" H 8383 4299 20  0000 C CNN
+F 2 "" H 7725 4125 60  0001 C CNN
+F 3 "" H 7725 4125 60  0001 C CNN
+	1    8350 4150
+	1    0    0    -1
+$EndComp
+$Comp
+L Device:D_Small D?
+U 1 1 6109C014
+P 8050 4400
+F 0 "D?" V 8096 4332 50  0000 R CNN
+F 1 "SOD-123" V 8005 4332 50  0000 R CNN
+F 2 "" V 8050 4400 50  0001 C CNN
+F 3 "~" V 8050 4400 50  0001 C CNN
+	1    8050 4400
+	0    -1   -1   0
+$EndComp
+Wire Wire Line
+	8300 4300 8050 4300
+Wire Wire Line
+	7000 3750 7300 3750
+Wire Wire Line
+	7300 3750 8050 3750
+Connection ~ 7300 3750
+Wire Wire Line
+	7000 4500 7300 4500
+Wire Wire Line
+	7300 4500 8050 4500
+Connection ~ 7300 4500
+Wire Wire Line
+	8500 4100 8500 3350
+Wire Wire Line
+	8500 3350 8500 3050
+Connection ~ 8500 3350
+Wire Wire Line
+	7750 4100 7750 3350
+Wire Wire Line
+	7750 3350 7750 3050
+Connection ~ 7750 3350
+Text GLabel 7000 3750 0    50   Input ~ 0
+ROW0
+Text GLabel 7000 4500 0    50   Input ~ 0
+ROW1
+Text GLabel 7750 3050 1    50   Input ~ 0
+COL0
+Text GLabel 8500 3050 1    50   Input ~ 0
+COL1
 $EndSCHEMATC
